File: boards/display_module/kicad/display_module.kicad_pcb (KiCad board)
At the start: 2 copper layers, 80 parts, among them IC1 ATMEGA328-P, P1 CONN_01X02, Q1 BC237, Q10 BC237, Q11 BC237, Q12 BC237, Q13 BC237, Q14 BC237, Q15 BC237, Q16 BC237, Q17 BC237, Q18 BC237, Q19 BC237, Q2 BC237, Q20 BC237, Q21 BC237, Q22 BC237, Q23 BC237, Q24 BC237, Q25 BC237, Q26 BC237, Q27 BC237, Q28 BC237, Q29 BC237, Q3 BC237, Q30 BC237, Q31 BC237, Q32 BC237, Q4 BC237, Q5 BC237, Q6 BC237, Q7 BC237, Q8 BC237, Q9 BC237, SW1 SW_PUSH, U1 74HC595, U2 74HC595, U3 74HC595, U4 74HC595, Y1 16M

Commit message: kicad update
Parts:
- removed PA1, PA2, PB1, PB2: CONN_01X12, Pin_Headers:Pin_Header_Straight_1x12
- removed R17, R18, R19, R20, R21, R22, R23, R24, R25, R26, R27, R28, R29, R30, R31, R32: R, Resistors_ThroughHole:Resistor_Horizontal_RM15mm
- added C5: 100n, Capacitors_ThroughHole:C_Disc_D3_P2.5, F.Cu at (172.7, 165.1)
- added C6: CP, Capacitors_ThroughHole:C_Radial_D5_L6_P2.5, F.Cu at (153.7, 165.1)
- added C7: 22p, Capacitors_ThroughHole:C_Disc_D3_P2.5, F.Cu at (166.4, 139.7)
- added C8: 22p, Capacitors_ThroughHole:C_Disc_D3_P2.5, F.Cu at (118.1, 184.2)
- added DISP1: LM23088A, my_footprints:LM23088A, F.Cu at (77.5, 77.5)
- added DISP2: LM23088A, my_footprints:LM23088A, F.Cu at (77.5, 135.9)
- added SW2: A, Buttons_Switches_ThroughHole:Push_E-Switch_KS01Q01, F.Cu at (212.1, 110.5)
- added SW3: B, Buttons_Switches_ThroughHole:Push_E-Switch_KS01Q01, F.Cu at (205.7, 76.2)
- added U5: SW10, my_footprints:SW10, F.Cu at (160.0, 152.4)
- added U6: SW10, my_footprints:SW10, F.Cu at (153.7, 152.4)
- C2: value CP -> 100n; footprint Capacitors_ThroughHole:C_Radial_D5_L6_P2.5 -> Capacitors_ThroughHole:C_Disc_D3_P2.5
- C3, C4: value 22p -> 100n
- Q1, Q10, Q11, Q12, Q13, Q14, Q15, Q16, Q2, Q3, Q4, Q5, Q6, Q7, Q8, Q9: value BC237 -> BC368; footprint TO_SOT_Packages_THT:TO-92_Inline_Wide -> TO_SOT_Packages_THT:TO-92_Inline_Narrow_Oval
- Q17, Q18, Q19, Q20, Q21, Q22, Q23, Q24, Q25, Q26, Q27, Q28, Q29, Q30, Q31, Q32: footprint TO_SOT_Packages_THT:TO-92_Inline_Wide -> TO_SOT_Packages_THT:TO-92_Inline_Narrow_Oval
- R1, R10, R11, R12, R13, R14, R15, R16, R2, R3, R4, R5, R6, R7, R8, R9: footprint Resistors_ThroughHole:Resistor_Horizontal_RM15mm -> Resistors_ThroughHole:Resistor_Horizontal_RM10mm
- SW1: value SW_PUSH -> RST
- moved Q28 201.2 mm to (125.7, 50.8)
- moved Q29 194.0 mm to (139.7, 45.7)
- moved Q27 184.6 mm to (133.3, 50.8)
- moved Q4 173.8 mm to (121.9, 170.2)
- moved Q19 172.3 mm to (148.6, 54.6)
- moved R4 169.4 mm to (119.4, 95.2)
- moved Q20 169.2 mm to (120.7, 68.6)
- moved Q18 167.2 mm to (141.0, 54.6)
- moved Q10 163.8 mm to (160.0, 45.7)
- moved Q13 163.4 mm to (152.4, 45.7)
- moved Q3 159.9 mm to (125.7, 162.6)
- moved R12 158.5 mm to (120.7, 59.7)
- moved Q15 157.5 mm to (166.4, 45.7)
- moved Q5 156.4 mm to (147.3, 174.0)
- moved R11 156.0 mm to (120.7, 77.5)
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Connections:
- C3 pad 1: GND -> VCC
- C3 pad 2: Net-(C3-Pad2) -> GND
- C4 pad 1: Net-(C4-Pad1) -> VCC
- IC1 pad 10: Net-(C4-Pad1) -> Net-(C8-Pad1)
- IC1 pad 11: Net-(IC1-Pad11) -> (no net)
- IC1 pad 12: Net-(IC1-Pad12) -> (no net)
- IC1 pad 13: Net-(IC1-Pad13) -> (no net)
- IC1 pad 14: Net-(IC1-Pad14) -> (no net)
- IC1 pad 2: Net-(IC1-Pad2) -> (no net)
- IC1 pad 26: Net-(IC1-Pad26) -> (no net)
- IC1 pad 3: Net-(IC1-Pad3) -> (no net)
- IC1 pad 4: Net-(IC1-Pad4) -> (no net)
- IC1 pad 5: Net-(IC1-Pad5) -> (no net)
- IC1 pad 6: Net-(IC1-Pad6) -> (no net)
- IC1 pad 9: Net-(C3-Pad2) -> Net-(C7-Pad2)
- Q1 pad 1: Net-(Q1-Pad1) -> GND
- Q1 pad 2: VCC -> Net-(DISP1-Pad18)
- Q10 pad 1: Net-(Q10-Pad1) -> GND
- Q10 pad 2: VCC -> Net-(DISP1-Pad2)
- Q11 pad 1: Net-(Q11-Pad1) -> GND
- Q11 pad 2: VCC -> Net-(DISP1-Pad4)
- Q12 pad 1: Net-(Q12-Pad1) -> GND
- Q12 pad 2: VCC -> Net-(DISP1-Pad5)
- Q13 pad 1: Net-(Q13-Pad1) -> GND
- Q13 pad 2: VCC -> Net-(DISP1-Pad7)
- Q14 pad 1: Net-(Q14-Pad1) -> GND
- Q14 pad 2: VCC -> Net-(DISP1-Pad8)
- Q15 pad 1: Net-(Q15-Pad1) -> GND
- Q15 pad 2: VCC -> Net-(DISP1-Pad10)
- Q16 pad 1: Net-(Q16-Pad1) -> GND
- Q16 pad 2: VCC -> Net-(DISP1-Pad11)
- Q17 pad 1: Net-(Q17-Pad1) -> VCC
- Q17 pad 2: Net-(PA1-Pad2) -> Net-(Q17-Pad2)
- Q17 pad 3: GND -> Net-(Q17-Pad3)
- Q18 pad 1: Net-(Q18-Pad1) -> VCC
- Q18 pad 2: Net-(PA1-Pad5) -> Net-(Q18-Pad2)
- Q18 pad 3: GND -> Net-(Q18-Pad3)
- Q19 pad 1: Net-(Q19-Pad1) -> VCC
- Q19 pad 2: Net-(PA1-Pad8) -> Net-(Q19-Pad2)
- Q19 pad 3: GND -> Net-(Q19-Pad3)
- Q2 pad 1: Net-(Q2-Pad1) -> GND
- Q2 pad 2: VCC -> Net-(DISP1-Pad24)
- Q20 pad 1: Net-(Q20-Pad1) -> VCC
- Q20 pad 2: Net-(PA1-Pad11) -> Net-(Q20-Pad2)
- Q20 pad 3: GND -> Net-(Q20-Pad3)
- Q21 pad 1: Net-(Q21-Pad1) -> VCC
- Q21 pad 2: Net-(PA2-Pad10) -> Net-(Q21-Pad2)
- Q21 pad 3: GND -> Net-(Q21-Pad3)
- Q22 pad 1: Net-(Q22-Pad1) -> VCC
- Q22 pad 2: Net-(PA2-Pad7) -> Net-(Q22-Pad2)
- Q22 pad 3: GND -> Net-(Q22-Pad3)
- Q23 pad 1: Net-(Q23-Pad1) -> VCC
- Q23 pad 2: Net-(PA2-Pad4) -> Net-(Q23-Pad2)
- Q23 pad 3: GND -> Net-(Q23-Pad3)
- Q24 pad 1: Net-(Q24-Pad1) -> VCC
- Q24 pad 2: Net-(PA2-Pad1) -> Net-(Q24-Pad2)
- Q24 pad 3: GND -> Net-(Q24-Pad3)
- Q25 pad 1: Net-(Q25-Pad1) -> VCC
- Q25 pad 2: Net-(PA1-Pad3) -> Net-(Q25-Pad2)
- Q25 pad 3: GND -> Net-(Q25-Pad3)
- Q26 pad 1: Net-(Q26-Pad1) -> VCC
- Q26 pad 2: Net-(PA1-Pad6) -> Net-(Q26-Pad2)
- Q26 pad 3: GND -> Net-(Q26-Pad3)
- Q27 pad 1: Net-(Q27-Pad1) -> VCC
- Q27 pad 2: Net-(PA1-Pad9) -> Net-(Q27-Pad2)
- Q27 pad 3: GND -> Net-(Q27-Pad3)
- Q28 pad 1: Net-(Q28-Pad1) -> VCC
- Q28 pad 2: Net-(PA1-Pad12) -> Net-(Q28-Pad2)
- Q28 pad 3: GND -> Net-(Q28-Pad3)
- Q29 pad 1: Net-(Q29-Pad1) -> VCC
- Q29 pad 2: Net-(PB2-Pad10) -> Net-(Q29-Pad2)
- Q29 pad 3: GND -> Net-(Q29-Pad3)
- Q3 pad 1: Net-(Q3-Pad1) -> GND
- Q3 pad 2: VCC -> Net-(DISP1-Pad23)
- Q30 pad 1: Net-(Q30-Pad1) -> VCC
- Q30 pad 2: Net-(PB2-Pad7) -> Net-(Q30-Pad2)
- Q30 pad 3: GND -> Net-(Q30-Pad3)
- Q31 pad 1: Net-(Q31-Pad1) -> VCC
- Q31 pad 2: Net-(PB2-Pad4) -> Net-(Q31-Pad2)
- Q31 pad 3: GND -> Net-(Q31-Pad3)
- Q32 pad 1: Net-(Q32-Pad1) -> VCC
- Q32 pad 2: Net-(PB2-Pad1) -> Net-(Q32-Pad2)
- Q32 pad 3: GND -> Net-(Q32-Pad3)
- Q4 pad 1: Net-(Q4-Pad1) -> GND
- Q4 pad 2: VCC -> Net-(DISP1-Pad21)
- Q5 pad 1: Net-(Q5-Pad1) -> GND
- Q5 pad 2: VCC -> Net-(DISP1-Pad20)
- Q6 pad 1: Net-(Q6-Pad1) -> GND
- Q6 pad 2: VCC -> Net-(DISP1-Pad17)
- Q7 pad 1: Net-(Q7-Pad1) -> GND
- Q7 pad 2: VCC -> Net-(DISP1-Pad15)
- Q8 pad 1: Net-(Q8-Pad1) -> GND
- Q8 pad 2: VCC -> Net-(DISP1-Pad14)
- Q9 pad 1: Net-(Q9-Pad1) -> GND
- Q9 pad 2: VCC -> Net-(DISP1-Pad1)
- R1 pad 2: Net-(Q1-Pad3) -> Net-(Q17-Pad3)
- R10 pad 2: Net-(Q10-Pad3) -> Net-(Q26-Pad3)
- R11 pad 2: Net-(Q11-Pad3) -> Net-(Q27-Pad3)
- R12 pad 2: Net-(Q12-Pad3) -> Net-(Q28-Pad3)
- R13 pad 2: Net-(Q13-Pad3) -> Net-(Q29-Pad3)
- R14 pad 2: Net-(Q14-Pad3) -> Net-(Q30-Pad3)
- R15 pad 2: Net-(Q15-Pad3) -> Net-(Q31-Pad3)
- R16 pad 2: Net-(Q16-Pad3) -> Net-(Q32-Pad3)
- R2 pad 2: Net-(Q2-Pad3) -> Net-(Q18-Pad3)
- R3 pad 2: Net-(Q3-Pad3) -> Net-(Q19-Pad3)
- R4 pad 2: Net-(Q4-Pad3) -> Net-(Q20-Pad3)
- R5 pad 2: Net-(Q5-Pad3) -> Net-(Q21-Pad3)
- R6 pad 2: Net-(Q6-Pad3) -> Net-(Q22-Pad3)
- R7 pad 2: Net-(Q7-Pad3) -> Net-(Q23-Pad3)
- R8 pad 2: Net-(Q8-Pad3) -> Net-(Q24-Pad3)
- R9 pad 2: Net-(Q9-Pad3) -> Net-(Q25-Pad3)
- U1 pad 1: Net-(R17-Pad2) -> Net-(Q19-Pad2)
- U1 pad 15: Net-(Q1-Pad1) -> Net-(Q17-Pad2)
- U1 pad 2: Net-(Q2-Pad1) -> Net-(Q21-Pad2)
- U1 pad 3: Net-(R18-Pad2) -> Net-(Q23-Pad2)
- U1 pad 4: Net-(Q3-Pad1) -> Net-(Q25-Pad2)
- U1 pad 5: Net-(R19-Pad2) -> Net-(Q27-Pad2)
- U1 pad 6: Net-(Q4-Pad1) -> Net-(Q29-Pad2)
- U1 pad 7: Net-(R20-Pad2) -> Net-(Q31-Pad2)
- U2 pad 1: Net-(R21-Pad2) -> Net-(Q3-Pad3)
- U2 pad 14: Net-(U1-Pad9) -> Net-(U2-Pad14)
- U2 pad 15: Net-(Q5-Pad1) -> Net-(Q2-Pad3)
- U2 pad 2: Net-(Q6-Pad1) -> Net-(Q4-Pad3)
- U2 pad 3: Net-(R22-Pad2) -> Net-(Q5-Pad3)
- U2 pad 4: Net-(Q7-Pad1) -> Net-(Q1-Pad3)
- U2 pad 5: Net-(R23-Pad2) -> Net-(Q6-Pad3)
- U2 pad 6: Net-(Q8-Pad1) -> Net-(Q7-Pad3)
- U2 pad 7: Net-(R24-Pad2) -> Net-(Q8-Pad3)
- U3 pad 1: Net-(R25-Pad2) -> Net-(Q10-Pad3)
- U3 pad 15: Net-(Q9-Pad1) -> Net-(Q9-Pad3)
- U3 pad 2: Net-(Q10-Pad1) -> Net-(Q11-Pad3)
- U3 pad 3: Net-(R26-Pad2) -> Net-(Q12-Pad3)
- U3 pad 4: Net-(Q11-Pad1) -> Net-(Q13-Pad3)
- U3 pad 5: Net-(R27-Pad2) -> Net-(Q14-Pad3)
- U3 pad 6: Net-(Q12-Pad1) -> Net-(Q15-Pad3)
- U3 pad 7: Net-(R28-Pad2) -> Net-(Q16-Pad3)
- U3 pad 9: Net-(U3-Pad9) -> (no net)
- U4 pad 1: Net-(R29-Pad2) -> Net-(Q20-Pad2)
- U4 pad 14: Net-(U3-Pad9) -> Net-(U1-Pad9)
- U4 pad 15: Net-(Q13-Pad1) -> Net-(Q18-Pad2)
- U4 pad 2: Net-(Q14-Pad1) -> Net-(Q22-Pad2)
- U4 pad 3: Net-(R30-Pad2) -> Net-(Q24-Pad2)
- U4 pad 4: Net-(Q15-Pad1) -> Net-(Q26-Pad2)
- U4 pad 5: Net-(R31-Pad2) -> Net-(Q28-Pad2)
- U4 pad 6: Net-(Q16-Pad1) -> Net-(Q30-Pad2)
- U4 pad 7: Net-(R32-Pad2) -> Net-(Q32-Pad2)
- U4 pad 9: Net-(U4-Pad9) -> Net-(U2-Pad14)
- Y1 pad 1: Net-(C3-Pad2) -> Net-(C7-Pad2)
- Y1 pad 2: Net-(C4-Pad1) -> Net-(C8-Pad1)
Other:
- board outline added: 58.4 x 148.6 mm
