File: boards/display_module/kicad/display_module.sch (KiCad schematic (older format))
At the start: 82 parts, among them IC1 ATMEGA328-P, P1 CONN_01X02, Q1 BC237, Q10 BC237, Q11 BC237, Q12 BC237, Q13 BC237, Q14 BC237, Q15 BC237, Q16 BC237, Q17 BC237, Q18 BC237, Q19 BC237, Q2 BC237, Q20 BC237, Q21 BC237, Q22 BC237, Q23 BC237, Q24 BC237, Q25 BC237, Q26 BC237, Q27 BC237, Q28 BC237, Q29 BC237, Q3 BC237, Q30 BC237, Q31 BC237, Q32 BC237, Q4 BC237, Q5 BC237, Q6 BC237, Q7 BC237, Q8 BC237, Q9 BC237, SW1 SW_PUSH, U1 74HC595, U2 74HC595, U3 74HC595, U4 74HC595, U5 SW10, U6 SW10, Y1 16M

Commit message: kicad update
Parts:
- removed PA1, PA2, PB1, PB2: CONN_01X12, Pin_Headers:Pin_Header_Straight_1x12, symbol CONN_01X12
- removed Q1, Q10, Q11, Q12, Q13, Q14, Q15, Q16, Q2, Q3, Q4, Q5, Q6, Q7, Q8, Q9: BC237, TO_SOT_Packages_THT:TO-92_Inline_Wide, symbol BC237
- removed R17, R18, R19, R20, R21, R22, R23, R24, R25, R26, R27, R28, R29, R30, R31, R32: R, Resistors_ThroughHole:Resistor_Horizontal_RM15mm, symbol R
- added C1, C2, C3, C5: 100n, Capacitors_ThroughHole:C_Disc_D3_P2.5, symbol C
- added DISP1, DISP2: LM23088A, my_footprints:LM23088A, symbol LM23088A
- added Q1, Q10, Q11, Q12, Q13, Q14, Q15, Q16, Q2, Q3, Q4, Q5, Q6, Q7, Q8, Q9: BC368, TO_SOT_Packages_THT:TO-92_Inline_Narrow_Oval, symbol Q_NPN_ECB
- added SW2: A, Buttons_Switches_ThroughHole:Push_E-Switch_KS01Q01, symbol SW_PUSH
- added SW3: B, Buttons_Switches_ThroughHole:Push_E-Switch_KS01Q01, symbol SW_PUSH
- Q17, Q18, Q19, Q20, Q21, Q22, Q23, Q24, Q25, Q26, Q27, Q28, Q29, Q30, Q31, Q32: footprint TO_SOT_Packages_THT:TO-92_Inline_Wide -> TO_SOT_Packages_THT:TO-92_Inline_Narrow_Oval
- R1, R10, R11, R12, R13, R14, R15, R16, R2, R3, R4, R5, R6, R7, R8, R9: footprint Resistors_ThroughHole:Resistor_Horizontal_RM15mm -> Resistors_ThroughHole:Resistor_Horizontal_RM10mm
- SW1: value SW_PUSH -> RST
- renumbered C1 to C4, C2 to C6, C3 to C7, C4 to C8, U4 to U3, U3 to U4
Connections:
- net GND: now also C1.2, C2.2, C3.2, C5.2, Q1.1 (E), Q10.1 (E), Q11.1 (E), Q12.1 (E), Q13.1 (E), Q14.1 (E), Q15.1 (E), Q16.1 (E), Q2.1 (E), Q3.1 (E), Q4.1 (E), Q5.1 (E), Q6.1 (E), Q7.1 (E), Q8.1 (E), Q9.1 (E), SW2.2, SW3.2; no longer Q17.3 (E), Q18.3 (E), Q19.3 (E), Q20.3 (E), Q21.3 (E), Q22.3 (E), Q23.3 (E), Q24.3 (E), Q25.3 (E), Q26.3 (E), Q27.3 (E), Q28.3 (E), Q29.3 (E), Q30.3 (E), Q31.3 (E), Q32.3 (E)
- net VCC: now also Q17.1 (C), Q18.1 (C), Q19.1 (C), Q20.1 (C), Q21.1 (C), Q22.1 (C), Q23.1 (C), Q24.1 (C), Q25.1 (C), Q26.1 (C), Q27.1 (C), Q28.1 (C), Q29.1 (C), Q30.1 (C), Q31.1 (C), Q32.1 (C), C1.1, C2.1, C3.1, C5.1
- net at IC1.27 ((PCINT12/SDA/ADC4)PC4): now also SW3.1
- net at IC1.28 ((PCINT13/SCL/ADC5)PC5): now also SW2.1
- net at U1.1 (QB): now also Q19.2 (B)
- net at U1.15 (QA): now also Q17.2 (B)
- net at U1.2 (QC): now also Q21.2 (B)
- net at U1.3 (QD): now also Q23.2 (B)
- net at U1.4 (QE): now also Q25.2 (B)
- net at U1.5 (QF): now also Q27.2 (B)
- net at U1.6 (QG): now also Q29.2 (B)
- net at U1.7 (QH): now also Q31.2 (B)
- net at U1.9 (~QH): now also U4.14 (SER); no longer U2.14 (SER)
- net at R1.2: now also Q17.3 (E)
- net at R1.1: now also DISP1.22 (A1)
- net at R4.1: now also DISP2.19 (A2)
- net at Q20.2 (B): now also U4.1 (QB)
- net at Q28.2 (B): now also U4.5 (QF)
- net at R2.1: now also DISP2.22 (A1)
- net at Q18.2 (B): now also U4.15 (QA)
- net at Q26.2 (B): now also U4.4 (QE)
- net at R3.1: now also DISP1.19 (A2)
- net at R2.2: now also Q18.3 (E)
- net at R3.2: now also Q19.3 (E)
- net at R4.2: now also Q20.3 (E)
- net at U2.1 (QB): now also Q3.3 (B)
- net at U2.15 (QA): now also Q2.3 (B)
- net at U2.2 (QC): now also Q4.3 (B)
- net at U2.3 (QD): now also Q5.3 (B)
- net at U2.4 (QE): now also Q1.3 (B)
- net at U2.5 (QF): now also Q6.3 (B)
- net at U2.6 (QG): now also Q7.3 (B)
- net at U2.7 (QH): now also Q8.3 (B)
- net at U2.9 (~QH): now also U3.14 (SER); no longer U4.14 (SER)
- net at R5.2: now also Q21.3 (E)
- net at R5.1: now also DISP1.16 (A3)
- net at Q24.2 (B): now also U4.3 (QD)
- net at R13.1: now also DISP1.9 (A7)
- net at R8.1: now also DISP2.13 (A4)
- net at R16.1: now also DISP2.12 (A8)
- net at R7.1: now also DISP1.13 (A4)
- net at R15.1: now also DISP1.12 (A8)
- net at Q22.2 (B): now also U4.2 (QC)
- net at R6.1: now also DISP2.16 (A3)
- net at R14.1: now also DISP2.9 (A7)
- net at R6.2: now also Q22.3 (E)
- net at R7.2: now also Q23.3 (E)
- net at R8.2: now also Q24.3 (E)
- net at U3.1 (QB): now also Q10.3 (B)
- net at U4.9 (~QH): now also U2.14 (SER); no longer U3.14 (SER)
- net at U3.15 (QA): now also Q9.3 (B)
- net at U3.2 (QC): now also Q11.3 (B)
- net at U3.3 (QD): now also Q12.3 (B)
- net at U3.4 (QE): now also Q13.3 (B)
- net at U3.5 (QF): now also Q14.3 (B)
- net at U3.6 (QG): now also Q15.3 (B)
- net at U3.7 (QH): now also Q16.3 (B)
- net at R13.2: now also Q29.3 (E)
- net at Q32.2 (B): now also U4.7 (QH)
- net at Q30.2 (B): now also U4.6 (QG)
- net at R14.2: now also Q30.3 (E)
- net at R15.2: now also Q31.3 (E)
- net at R16.2: now also Q32.3 (E)
- net at R9.2: now also Q25.3 (E)
- net at R9.1: now also DISP1.3 (A5)
- net at R10.2: now also Q26.3 (E)
- net at R10.1: now also DISP2.3 (A5)
- net at R11.2: now also Q27.3 (E)
- net at R11.1: now also DISP1.6 (A6)
- net at R12.2: now also Q28.3 (E)
- net at R12.1: now also DISP2.6 (A6)
- new net: DISP1.1 (KR4), DISP2.1 (KR4), Q9.2 (C)
- new net: DISP1.10 (KG8), DISP2.10 (KG8), Q15.2 (C)
- new net: DISP1.11 (KR8), DISP2.11 (KR8), Q16.2 (C)
- new net: DISP1.14 (KG5), DISP2.14 (KG5), Q8.2 (C)
- new net: DISP1.15 (KG4), DISP2.15 (KG4), Q7.2 (C)
- new net: DISP1.17 (KR3), DISP2.17 (KR3), Q6.2 (C)
- new net: DISP1.18 (KG3), DISP2.18 (KG3), Q1.2 (C)
- new net: DISP1.2 (KR5), DISP2.2 (KR5), Q10.2 (C)
- new net: DISP1.20 (KR2), DISP2.20 (KR2), Q5.2 (C)
- new net: DISP1.21 (KG2), DISP2.21 (KG2), Q4.2 (C)
- new net: DISP1.23 (KR1), DISP2.23 (KR1), Q3.2 (C)
- new net: DISP1.24 (KG1), DISP2.24 (KG1), Q2.2 (C)
- new net: DISP1.4 (KG6), DISP2.4 (KG6), Q11.2 (C)
- new net: DISP1.5 (KR6), DISP2.5 (KR6), Q12.2 (C)
- new net: DISP1.7 (KG7), DISP2.7 (KG7), Q13.2 (C)
- new net: DISP1.8 (KR7), DISP2.8 (KR7), Q14.2 (C)
- no-connect marks 23 -> 21
Other:
- moved on the sheet: SW1, U2, U3, U4

Commit message: kicad work
Parts:
- removed C3, C5: 100n, Capacitors_ThroughHole:C_Disc_D3_P2.5, symbol C
- removed Q1, Q10, Q11, Q12, Q13, Q14, Q15, Q16, Q2, Q3, Q4, Q5, Q6, Q7, Q8, Q9: BC368, TO_SOT_Packages_THT:TO-92_Inline_Narrow_Oval, symbol Q_NPN_ECB
- removed Q17, Q18, Q19, Q20, Q21, Q22, Q23, Q24, Q25, Q26, Q27, Q28, Q29, Q30, Q31, Q32: BC237, TO_SOT_Packages_THT:TO-92_Inline_Narrow_Oval, symbol BC237
- removed R10, R11, R12, R13, R14, R15, R16, R9: 10, Resistors_ThroughHole:Resistor_Horizontal_RM10mm, symbol R
- removed SW1: RST, Buttons_Switches_ThroughHole:Push_E-Switch_KS01Q01, symbol SW_PUSH
- removed SW2: A, Buttons_Switches_ThroughHole:Push_E-Switch_KS01Q01, symbol SW_PUSH
- removed SW3: B, Buttons_Switches_ThroughHole:Push_E-Switch_KS01Q01, symbol SW_PUSH
- removed U1, U2, U3, U4: 74HC595, Housings_DIP:DIP-16_W7.62mm, symbol 74HC595
- added Q1, Q2, Q3, Q4, Q5, Q6, Q7, Q8: NDP6020P, TO_SOT_Packages_THT:TO-220_Vertical, symbol NDP6020P
- added U1, U2: TLC5940NT, Housings_DIP:DIP-28_W7.62mm, symbol TLC5940NT
- C1, C2: footprint Capacitors_ThroughHole:C_Disc_D3_P2.5 -> Capacitors_ThroughHole:C_Disc_D3.0mm_W1.6mm_P2.50mm
- C3: renamed from C4; footprint Capacitors_ThroughHole:C_Disc_D3_P2.5 -> Capacitors_ThroughHole:C_Disc_D3.0mm_W1.6mm_P2.50mm
- C4: renamed from C6; value CP -> 10uF; footprint Capacitors_ThroughHole:C_Radial_D5_L6_P2.5 -> Capacitors_ThroughHole:CP_Radial_D5.0mm_P2.50mm
- C5: renamed from C7; footprint Capacitors_ThroughHole:C_Disc_D3_P2.5 -> Capacitors_ThroughHole:C_Disc_D3.0mm_W1.6mm_P2.50mm
- C6: renamed from C8; footprint Capacitors_ThroughHole:C_Disc_D3_P2.5 -> Capacitors_ThroughHole:C_Disc_D3.0mm_W1.6mm_P2.50mm
- R1, R2, R4, R6, R8: value 10 -> 380; footprint Resistors_ThroughHole:Resistor_Horizontal_RM10mm -> Resistors_ThroughHole:R_Axial_DIN0204_L3.6mm_D1.6mm_P5.08mm_Horizontal
- R3, R5, R7: value 10 -> 190; footprint Resistors_ThroughHole:Resistor_Horizontal_RM10mm -> Resistors_ThroughHole:R_Axial_DIN0204_L3.6mm_D1.6mm_P5.08mm_Horizontal
- Y1: footprint Crystals:Crystal_HC48-U_Vertical -> Crystals:Crystal_HC50_Vertical
- renumbered U6 to SPI_IN1, U5 to SPI_OUT1
Connections:
- net GND: now also R1.2, R2.2, R4.2, R6.2, R8.2, SPI_IN1.5 (GND), SPI_OUT1.5 (GND), U1.19 (DCPRG), U1.22 (GND), U1.27 (VPRG), U2.19 (DCPRG), U2.22 (GND), U2.27 (VPRG); no longer SPI_IN1.10, SPI_OUT1.10
- net VCC: now also R3.2, R5.2, R7.2, Q1.3 (S), Q2.3 (S), Q3.3 (S), Q4.3 (S), Q5.3 (S), Q6.3 (S), Q7.3 (S), Q8.3 (S), U1.21 (VCC), U2.21 (VCC)
- net at IC1.11 ((PCINT21/OC0B/T1)PD5): now also Q6.1 (G)
- net at IC1.12 ((PCINT22/OC0A/AIN0)PD6): now also Q7.1 (G)
- net at IC1.13 ((PCINT23/AIN1)PD7): now also Q8.1 (G)
- net at IC1.14 ((PCINT0/CLKO/ICP1)PB0): now also SPI_OUT1.7 (SS_DISP)
- net at IC1.15 ((PCINT1/OC1A)PB1): now also U1.18 (GSCLK), U2.18 (GSCLK); no longer SPI_OUT1.7 (SS_DISP)
- net at IC1.16 ((PCINT2/OC1B/~SS~)PB2), SPI_IN1.7 (SS_DISP): now also R6.1, R7.1
- net at IC1.17 ((PCINT3/OC2A/MOSI)PB3), SPI_IN1.4 (MOSI), SPI_OUT1.4 (MOSI): now also R4.1, R5.1
- net at IC1.19 ((PCINT5/SCK)PB5), SPI_IN1.2 (SCK), SPI_OUT1.2 (SCK): now also R2.1, R3.1
- net at IC1.2 ((PCINT16/RXD)PD0): now also Q1.1 (G)
- net at IC1.25 ((PCINT10/ADC2)PC2): now also U1.23 (BLANK), U2.23 (BLANK)
- net at IC1.26 ((PCINT11/ADC3)PC3): now also U1.24 (XLAT), U2.24 (XLAT)
- net at IC1.27 ((PCINT12/SDA/ADC4)PC4): now also U1.25 (SCLK), U2.25 (SCLK)
- net at IC1.28 ((PCINT13/SCL/ADC5)PC5): now also U1.26 (SIN)
- net at IC1.3 ((PCINT17/TXD)PD1): now also Q2.1 (G)
- net at IC1.4 ((PCINT18/INT0)PD2): now also Q3.1 (G)
- net at IC1.5 ((PCINT19/OC2B/INT1)PD3): now also Q4.1 (G)
- net at IC1.6 ((PCINT20/XCK/T0)PD4): now also Q5.1 (G)
- net at DISP1.1 (KR4): now also U1.8 (OUT8); no longer DISP2.1 (KR4)
- net at DISP1.10 (KG8): now also U1.14 (OUT14); no longer DISP2.10 (KG8)
- net at DISP1.11 (KR8): now also U1.15 (OUT15); no longer DISP2.11 (KR8)
- net at DISP1.12 (A8): now also DISP2.12 (A8), Q8.2 (D)
- net at DISP1.13 (A4): now also DISP2.13 (A4), Q4.2 (D); no longer R7.1
- net at DISP1.14 (KG5): now also U1.7 (OUT7); no longer DISP2.14 (KG5)
- net at DISP1.15 (KG4): now also U1.6 (OUT6); no longer DISP2.15 (KG4)
- net at DISP1.16 (A3): now also DISP2.16 (A3), Q3.2 (D); no longer R5.1
- net at DISP1.17 (KR3): now also U1.5 (OUT5); no longer DISP2.17 (KR3)
- net at DISP1.18 (KG3): now also U1.4 (OUT4); no longer DISP2.18 (KG3)
- net at DISP1.19 (A2): now also DISP2.19 (A2), Q2.2 (D); no longer R3.1
- net at DISP1.2 (KR5): now also U1.9 (OUT9); no longer DISP2.2 (KR5)
- net at DISP1.20 (KR2): now also U1.3 (OUT3); no longer DISP2.20 (KR2)
- net at DISP1.21 (KG2): now also U1.2 (OUT2); no longer DISP2.21 (KG2)
- net at DISP1.22 (A1): now also DISP2.22 (A1), Q1.2 (D); no longer R1.1
- net at DISP1.23 (KR1): now also U1.1 (OUT1); no longer DISP2.23 (KR1)
- net at DISP1.24 (KG1): now also U1.28 (OUT0); no longer DISP2.24 (KG1)
- net at DISP1.3 (A5): now also DISP2.3 (A5), Q5.2 (D)
- net at DISP1.4 (KG6): now also U1.10 (OUT10); no longer DISP2.4 (KG6)
- net at DISP1.5 (KR6): now also U1.11 (OUT11); no longer DISP2.5 (KR6)
- net at DISP1.6 (A6): now also DISP2.6 (A6), Q6.2 (D)
- net at DISP1.7 (KG7): now also U1.12 (OUT12); no longer DISP2.7 (KG7)
- net at DISP1.8 (KR7): now also U1.13 (OUT13); no longer DISP2.8 (KR7)
- net at DISP1.9 (A7): now also DISP2.9 (A7), Q7.2 (D)
- net at R8.1: now also U2.20 (IREF); no longer DISP2.13 (A4)
- new net: DISP2.23 (KR1), U2.1 (OUT1)
- new net: DISP2.4 (KG6), U2.10 (OUT10)
- new net: DISP2.5 (KR6), U2.11 (OUT11)
- new net: DISP2.7 (KG7), U2.12 (OUT12)
- new net: DISP2.8 (KR7), U2.13 (OUT13)
- new net: DISP2.10 (KG8), U2.14 (OUT14)
- new net: DISP2.11 (KR8), U2.15 (OUT15)
- new net: DISP2.21 (KG2), U2.2 (OUT2)
- new net: U1.17 (SOUT), U2.26 (SIN)
- new net: DISP2.24 (KG1), U2.28 (OUT0)
- new net: DISP2.20 (KR2), U2.3 (OUT3)
- new net: DISP2.18 (KG3), U2.4 (OUT4)
- new net: DISP2.17 (KR3), U2.5 (OUT5)
- new net: DISP2.15 (KG4), U2.6 (OUT6)
- new net: DISP2.14 (KG5), U2.7 (OUT7)
- new net: DISP2.1 (KR4), U2.8 (OUT8)
- new net: DISP2.2 (KR5), U2.9 (OUT9)
- new net: R1.1, U1.20 (IREF)
- no-connect marks 21 -> 16

Commit message: WIP: display module PCB design v2.1
Parts:
- added J1: SELFTEST, symbol CONN_01X02
- added J2: AUX, symbol CONN_01X02
- added R10, R11, R12, R13, R14, R15, R16, R9: 10k, Resistors_ThroughHole:R_Axial_DIN0204_L3.6mm_D1.6mm_P5.08mm_Horizontal, symbol R
- added U3: ICSP, symbol ICSP
- P1: value CONN_01X02 -> POWER
Connections:
- net GND: now also J1.2 (P2), J2.2 (P2), U3.6 (GND)
- net VCC: now also R10.1, R11.1, R12.1, R13.1, R14.1, R15.1, R16.1, R9.1, U3.2 (VCC)
- net at IC1.1 ((PCINT14/~RESET~)PC6): now also U3.5 (RST)
- net at IC1.11 ((PCINT21/OC0B/T1)PD5), Q6.1 (G): now also R14.2
- net at IC1.12 ((PCINT22/OC0A/AIN0)PD6), Q7.1 (G): now also R15.2
- net at IC1.13 ((PCINT23/AIN1)PD7), Q8.1 (G): now also R16.2
- net at IC1.17 ((PCINT3/OC2A/MOSI)PB3), R4.1, R5.1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: now also U3.4 (MOSI)
- net at IC1.18 ((PCINT4/MISO)PB4), SPI_IN1.3 (MISO), SPI_OUT1.3 (MISO): now also U3.1 (MISO)
- net at IC1.19 ((PCINT5/SCK)PB5), R2.1, R3.1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: now also U3.3 (SCK)
- net at IC1.2 ((PCINT16/RXD)PD0), Q1.1 (G): now also R9.2
- net at IC1.23 ((PCINT8/ADC0)PC0): now also J1.1 (P1)
- net at IC1.24 ((PCINT9/ADC1)PC1): now also J2.1 (P1)
- net at IC1.3 ((PCINT17/TXD)PD1), Q2.1 (G): now also R10.2
- net at IC1.4 ((PCINT18/INT0)PD2), Q3.1 (G): now also R11.2
- net at IC1.5 ((PCINT19/OC2B/INT1)PD3), Q4.1 (G): now also R12.2
- net at IC1.6 ((PCINT20/XCK/T0)PD4), Q5.1 (G): now also R13.2
- no-connect marks 16 -> 13

Commit message: WIP: display module PCB design v2.1
Parts:
- J1, J2: footprint (none) -> my_footprints:PINS1x2
- R1, R10, R11, R12, R13, R14, R15, R16, R2, R3, R4, R5, R6, R7, R8, R9: footprint Resistors_ThroughHole:R_Axial_DIN0204_L3.6mm_D1.6mm_P5.08mm_Horizontal -> Resistors_ThroughHole:R_Axial_DIN0204_L3.6mm_D1.6mm_P7.62mm_Horizontal
- U3: footprint (none) -> my_footprints:PINS3x2
Changed lines of the file:
@@
 F 0 "R1" V 3730 7400 50  0000 C CNN
 F 1 "380" V 3650 7400 50  0000 C CNN
-F 2 "Resistors_ThroughHole:R_Axial_DIN0204_L3.6mm_D1.6mm_P5.08mm_Horizontal" V 3580 7400 50  0001 C CNN
+F 2 "Resistors_ThroughHole:R_Axial_DIN0204_L3.6mm_D1.6mm_P7.62mm_Horizontal" V 3580 7400 50  0001 C CNN
 F 3 "" H 3650 7400 50  0001 C CNN
 	1    3650 7400
@@
 F 0 "R8" V 8230 7400 50  0000 C CNN
 F 1 "380" V 8150 7400 50  0000 C CNN
-F 2 "Resistors_ThroughHole:R_Axial_DIN0204_L3.6mm_D1.6mm_P5.08mm_Horizontal" V 8080 7400 50  0001 C CNN
+F 2 "Resistors_ThroughHole:R_Axial_DIN0204_L3.6mm_D1.6mm_P7.62mm_Horizontal" V 8080 7400 50  0001 C CNN
 F 3 "" H 8150 7400 50  0001 C CNN
 	1    8150 7400
@@
 F 0 "R2" V 5530 1900 50  0000 C CNN
 F 1 "380" V 5450 1900 50  0000 C CNN
-F 2 "Resistors_ThroughHole:R_Axial_DIN0204_L3.6mm_D1.6mm_P5.08mm_Horizontal" V 5380 1900 50  0001 C CNN
+F 2 "Resistors_ThroughHole:R_Axial_DIN0204_L3.6mm_D1.6mm_P7.62mm_Horizontal" V 5380 1900 50  0001 C CNN
 F 3 "" H 5450 1900 50  0001 C CNN
 	1    5450 1900
@@
 F 0 "R3" V 5730 1900 50  0000 C CNN
 F 1 "190" V 5650 1900 50  0000 C CNN
-F 2 "Resistors_ThroughHole:R_Axial_DIN0204_L3.6mm_D1.6mm_P5.08mm_Horizontal" V 5580 1900 50  0001 C CNN
+F 2 "Resistors_ThroughHole:R_Axial_DIN0204_L3.6mm_D1.6mm_P7.62mm_Horizontal" V 5580 1900 50  0001 C CNN
 F 3 "" H 5650 1900 50  0001 C CNN
 	1    5650 1900
@@
 F 0 "R4" V 5980 1900 50  0000 C CNN
 F 1 "380" V 5900 1900 50  0000 C CNN
-F 2 "Resistors_ThroughHole:R_Axial_DIN0204_L3.6mm_D1.6mm_P5.08mm_Horizontal" V 5830 1900 50  0001 C CNN
+F 2 "Resistors_ThroughHole:R_Axial_DIN0204_L3.6mm_D1.6mm_P7.62mm_Horizontal" V 5830 1900 50  0001 C CNN
 F 3 "" H 5900 1900 50  0001 C CNN
 	1    5900 1900
@@
 F 0 "R5" V 6180 1900 50  0000 C CNN
 F 1 "190" V 6100 1900 50  0000 C CNN
-F 2 "Resistors_ThroughHole:R_Axial_DIN0204_L3.6mm_D1.6mm_P5.08mm_Horizontal" V 6030 1900 50  0001 C CNN
+F 2 "Resistors_ThroughHole:R_Axial_DIN0204_L3.6mm_D1.6mm_P7.62mm_Horizontal" V 6030 1900 50  0001 C CNN
 F 3 "" H 6100 1900 50  0001 C CNN
 	1    6100 1900
@@
 F 0 "R6" V 6530 1900 50  0000 C CNN
 F 1 "380" V 6450 1900 50  0000 C CNN
-F 2 "Resistors_ThroughHole:R_Axial_DIN0204_L3.6mm_D1.6mm_P5.08mm_Horizontal" V 6380 1900 50  0001 C CNN
+F 2 "Resistors_ThroughHole:R_Axial_DIN0204_L3.6mm_D1.6mm_P7.62mm_Horizontal" V 6380 1900 50  0001 C CNN
 F 3 "" H 6450 1900 50  0001 C CNN
 	1    6450 1900
@@
 F 0 "R7" V 6730 1900 50  0000 C CNN
 F 1 "190" V 6650 1900 50  0000 C CNN
-F 2 "Resistors_ThroughHole:R_Axial_DIN0204_L3.6mm_D1.6mm_P5.08mm_Horizontal" V 6580 1900 50  0001 C CNN
+F 2 "Resistors_ThroughHole:R_Axial_DIN0204_L3.6mm_D1.6mm_P7.62mm_Horizontal" V 6580 1900 50  0001 C CNN
 F 3 "" H 6650 1900 50  0001 C CNN
 	1    6650 1900
@@
 F 0 "R10" V 6080 3050 50  0000 C CNN
 F 1 "10k" V 6000 3050 50  0000 C CNN
-F 2 "Resistors_ThroughHole:R_Axial_DIN0204_L3.6mm_D1.6mm_P5.08mm_Horizontal" V 5930 3050 50  0001 C CNN
+F 2 "Resistors_ThroughHole:R_Axial_DIN0204_L3.6mm_D1.6mm_P7.62mm_Horizontal" V 5930 3050 50  0001 C CNN
 F 3 "" H 6000 3050 50  0001 C CNN
 	1    6000 3050
@@
 F 0 "R9" V 5180 3050 50  0000 C CNN
 F 1 "10k" V 5100 3050 50  0000 C CNN
-F 2 "Resistors_ThroughHole:R_Axial_DIN0204_L3.6mm_D1.6mm_P5.08mm_Horizontal" V 5030 3050 50  0001 C CNN
+F 2 "Resistors_ThroughHole:R_Axial_DIN0204_L3.6mm_D1.6mm_P7.62mm_Horizontal" V 5030 3050 50  0001 C CNN
 F 3 "" H 5100 3050 50  0001 C CNN
 	1    5100 3050
@@
 F 0 "R11" V 6980 3050 50  0000 C CNN
 F 1 "10k" V 6900 3050 50  0000 C CNN
-F 2 "Resistors_ThroughHole:R_Axial_DIN0204_L3.6mm_D1.6mm_P5.08mm_Horizontal" V 6830 3050 50  0001 C CNN
+F 2 "Resistors_ThroughHole:R_Axial_DIN0204_L3.6mm_D1.6mm_P7.62mm_Horizontal" V 6830 3050 50  0001 C CNN
 F 3 "" H 6900 3050 50  0001 C CNN
 	1    6900 3050
@@
 F 0 "R12" V 7880 3050 50  0000 C CNN
 F 1 "10k" V 7800 3050 50  0000 C CNN
-F 2 "Resistors_ThroughHole:R_Axial_DIN0204_L3.6mm_D1.6mm_P5.08mm_Horizontal" V 7730 3050 50  0001 C CNN
+F 2 "Resistors_ThroughHole:R_Axial_DIN0204_L3.6mm_D1.6mm_P7.62mm_Horizontal" V 7730 3050 50  0001 C CNN
 F 3 "" H 7800 3050 50  0001 C CNN
 	1    7800 3050
@@
 F 0 "R13" V 8780 3050 50  0000 C CNN
 F 1 "10k" V 8700 3050 50  0000 C CNN
-F 2 "Resistors_ThroughHole:R_Axial_DIN0204_L3.6mm_D1.6mm_P5.08mm_Horizontal" V 8630 3050 50  0001 C CNN
+F 2 "Resistors_ThroughHole:R_Axial_DIN0204_L3.6mm_D1.6mm_P7.62mm_Horizontal" V 8630 3050 50  0001 C CNN
 F 3 "" H 8700 3050 50  0001 C CNN
 	1    8700 3050
@@
 F 0 "R14" V 9680 3050 50  0000 C CNN
 F 1 "10k" V 9600 3050 50  0000 C CNN
-F 2 "Resistors_ThroughHole:R_Axial_DIN0204_L3.6mm_D1.6mm_P5.08mm_Horizontal" V 9530 3050 50  0001 C CNN
+F 2 "Resistors_ThroughHole:R_Axial_DIN0204_L3.6mm_D1.6mm_P7.62mm_Horizontal" V 9530 3050 50  0001 C CNN
 F 3 "" H 9600 3050 50  0001 C CNN
 	1    9600 3050
@@
 F 0 "R15" V 10580 3050 50  0000 C CNN
 F 1 "10k" V 10500 3050 50  0000 C CNN
-F 2 "Resistors_ThroughHole:R_Axial_DIN0204_L3.6mm_D1.6mm_P5.08mm_Horizontal" V 10430 3050 50  0001 C CNN
+F 2 "Resistors_ThroughHole:R_Axial_DIN0204_L3.6mm_D1.6mm_P7.62mm_Horizontal" V 10430 3050 50  0001 C CNN
 F 3 "" H 10500 3050 50  0001 C CNN
 	1    10500 3050
@@
 F 0 "R16" V 11480 3050 50  0000 C CNN
 F 1 "10k" V 11400 3050 50  0000 C CNN
-F 2 "Resistors_ThroughHole:R_Axial_DIN0204_L3.6mm_D1.6mm_P5.08mm_Horizontal" V 11330 3050 50  0001 C CNN
+F 2 "Resistors_ThroughHole:R_Axial_DIN0204_L3.6mm_D1.6mm_P7.62mm_Horizontal" V 11330 3050 50  0001 C CNN
 F 3 "" H 11400 3050 50  0001 C CNN
 	1    11400 3050
@@
 F 0 "U3" H 8050 1300 60  0000 C CNN
 F 1 "ICSP" H 7600 1300 60  0000 C CNN
-F 2 "" H 7620 860 60  0001 C CNN
+F 2 "my_footprints:PINS3x2" H 7620 860 60  0001 C CNN
 F 3 "" H 7620 860 60  0001 C CNN
 	1    7750 1000
@@
 F 0 "J1" H 4550 2150 50  0000 C CNN
 F 1 "SELFTEST" V 4650 2000 50  0000 C CNN
-F 2 "" H 4550 2000 50  0001 C CNN
+F 2 "my_footprints:PINS1x2" H 4550 2000 50  0001 C CNN
 F 3 "" H 4550 2000 50  0001 C CNN
 	1    4550 2000
@@
 F 0 "J2" H 5050 2150 50  0000 C CNN
 F 1 "AUX" V 5150 2000 50  0000 C CNN
-F 2 "" H 5050 2000 50  0001 C CNN
+F 2 "my_footprints:PINS1x2" H 5050 2000 50  0001 C CNN
 F 3 "" H 5050 2000 50  0001 C CNN
 	1    5050 2000
